File: pcb/main-controller/main-controller.kicad_sch (KiCad schematic)
At the start: 20 parts, among them J1 ICM20948 - IMU, J2 Current-sensor, J3 Battery charge, J4 Conn_01x02_Pin, J5 Conn_01x02_Pin, J6 Conn_01x02_Pin, J7 Conn_01x02_Pin, J8 M1, J9 M2, SW1 SW_SPST

Commit message: vault backup: 2026-10-16 15:18:46
Parts:
- J4: value Conn_01x02_Pin -> B3
- J5: value Conn_01x02_Pin -> B4
- J6: value Conn_01x02_Pin -> B1
- J7: value Conn_01x02_Pin -> B2
Connections:
- net VBUS: now reaches J4.1 (Pin_1)
- net VBUS: now also J3.1 (Pin_1)
- net at J4.2 (Pin_2), J5.1 (Pin_1): now also J3.2 (Pin_2)
- net at J6.1 (Pin_1): now also J3.5 (Pin_5), J7.2 (Pin_2)
- net VCC: now reaches J6.2 (Pin_2)
- net VCC: now also J3.6 (Pin_6), SW1.1 (A)
- net at SW1.2 (B): now also A1.VIN
- net +3.3V: now reaches J1.1 (Pin_1)
- net +3.3V: now also A1.3V3 (3.3V)
- net GND: now reaches J1.5 (Pin_5)
- net GND: now also A1.GND1 (GND), A1.GND2 (GND), J3.3 (Pin_3), J3.4 (Pin_4), J5.2 (Pin_2), J7.1 (Pin_1)
- net VDD: now reaches J2.8 (Pin_8)
